File: hardware/sao-wall.kicad_sch (KiCad schematic)
At the start: 40 parts, among them CON1 AVR-ISP-6, J1 PMOD-2x6-MALE, J2 PMOD-2x6-FEMALE, Q1 PMBT2907A_PNP_500mA, Q2 PMBT2907A_PNP_500mA, Q3 PMBT2907A_PNP_500mA, U1 ATmega32U4-MU, U2 TLV62569DBVR, X1 16MHz, X2 A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

Commit message: hardware: move to QFP cpu package, Dec2022 release
Parts:
- U1: footprint tom-semiconductors:QFN-44-1EP_7x7mm_P0.5mm_EP5.15x5.15mm -> tom-semiconductors:TQFP-44_10x10mm_P0.8mm
Changed lines of the file:
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@@
     (property "Reference" "U1" (id 0) (at 189.23 118.11 0))
     (property "Value" "ATmega32U4-MU" (id 1) (at 210.82 118.11 0))
-    (property "Footprint" "tom-semiconductors:QFN-44-1EP_7x7mm_P0.5mm_EP5.15x5.15mm" (id 2) (at 200.66 73.66 0)
+    (property "Footprint" "tom-semiconductors:TQFP-44_10x10mm_P0.8mm" (id 2) (at 200.66 73.66 0)
       (effects (font (size 1.27 1.27) italic) hide)
     )
@@
     )
     (path "/00000000-0000-0000-0000-00005f895d6d"
-      (reference "U1") (unit 1) (value "ATmega32U4-MU") (footprint "tom-semiconductors:QFN-44-1EP_7x7mm_P0.5mm_EP5.15x5.15mm")
+      (reference "U1") (unit 1) (value "ATmega32U4-MU") (footprint "tom-semiconductors:TQFP-44_10x10mm_P0.8mm")
     )
     (path "/00000000-0000-0000-0000-00005fa51e67"
